Commit message: now

File: src/rain_arm_description/urdf/rain_arm.urdf.xacro (robot description, xacro)
@@ -22,5 +22,5 @@
             <origin xyz="-0.39 -0.39 -0.56" rpy="0.0 0.0 0.0"/>
             <geometry>
-                <mesh filename="package://rain_arm_description/meshes/-.STL" scale="0.01 0.01 0.01"/>
+                <mesh filename="package://rain_arm_description/meshes/base_plate.STL" scale="0.01 0.01 0.01"/>
             </geometry>
         </visual>

Commit message: now

File: src/rain_arm_description/urdf/rain_arm.urdf.xacro (robot description, xacro)
@@ -33,3 +33,77 @@
         <limit lower="-${PI/2}" upper="${PI/2}" effort="${effort}" velocity="${velocity}"/>
     </joint>
+    <link name="forward_drive_arm">
+        <visual>
+            <origin rpy="0.0 -${PI/2} ${PI/2}" xyz="0.19 0.06 -0.08"/>
+            <geometry>
+                <mesh filename="package://rain_arm_description/meshes/forward_drive_arm.STL" scale="0.01 0.01 0.01"/>
+            </geometry>
+        </visual>
+    </link>
+    <joint name="base_plate_forward_drive_arm" type="revolute">
+        <parent link="base_plate"/>
+        <child link="forward_drive_arm"/>
+        <origin xyz="-0.02 0.0 0.35" rpy="0.0 0.0 0.0"/>
+        <axis xyz="1.0 0.0 0.0"/>
+        <limit lower="-${PI/2}" upper="${PI/2}" effort="${effort}" velocity="${velocity}"/>
+    </joint>
+    <link name="horizontal_arm">
+        <visual>
+            <origin rpy="${PI/2} 0.0 ${PI/2}" xyz="-0.03 -0.4 -0.06"/>
+            <geometry>
+                <mesh filename="package://rain_arm_description/meshes/horizontal_arm.STL" scale="0.01 0.01 0.01"/>
+            </geometry>
+        </visual>
+    </link>
+    <joint name="forward_drive_arm_horizontal_arm" type="revolute">
+        <parent link="forward_drive_arm"/>
+        <child link="horizontal_arm"/>
+        <limit lower="-${PI/2}" upper="${PI/2}" effort="${effort}" velocity="${velocity}"/>
+        <axis xyz="1.0 0.0 0.0"/>
+        <origin xyz="0.0 0.0 0.8" rpy="0.0 0.0 0.0"/>
+    </joint>
+    <link name="claw_base">
+        <visual>
+            <origin xyz="0.0 -0.05 -0.15" rpy="0.0 0.0 ${PI/2}"/>
+            <geometry>
+                <mesh filename="package://rain_arm_description/meshes/claw_support.STL" scale="0.01 0.01 0.01"/>
+            </geometry>
+        </visual>
+    </link>
+        <joint name="horizontal_arm_claw_base" type="fixed">
+            <parent link="horizontal_arm"/>
+            <child link="claw_base"/>
+            <origin xyz="0.0 0.82 0.0" rpy="0.0 0.0 0.0"/>
+        </joint>
+        <link name="gripper_right">
+            <visual>
+                <origin xyz="-0.1 0.5 -0.1" rpy="0.0 0.0 -${PI/2}"/>
+                <geometry>
+                    <mesh filename="package://rain_arm_description/meshes/right_finger.STL" scale="0.01 0.01 0.01"/>
+                </geometry>
+            </visual>
+        </link>
+        <link name="gripper_left">
+            <visual>
+                <origin xyz="-0.04 0.5 -0.1" rpy="0.0 0.0 -${PI/2}"/>
+                <geometry>
+                    <mesh filename="package://rain_arm_description/meshes/left_finger.STL" scale="0.01 0.01 0.01"/>
+                </geometry>
+            </visual>
+        </link>
+    <joint name="claw_base_gripper_right" type="revolute">
+        <parent link="claw_base"/>
+        <child link="gripper_right"/>
+        <axis xyz="0.0 0.0 1.0"/>
+        <origin xyz="-0.04 0.13 -0.1" rpy="0.0 0.0 0.0"/>
+        <limit lower="-${PI/2}" upper="0.0" effort="${effort}" velocity="${velocity}"/>
+    </joint>
+    <joint name="claw_base_gripper_left" type="revolute">
+        <parent link="claw_base"/>
+        <child link="gripper_left"/>
+        <axis xyz="0.0 0.0 1.0"/>
+        <origin xyz="-0.22 0.13 -0.1" rpy="0.0 0.0 0.0"/>
+        <mimic joint = "claw_base_gripper_right" multiplier = "-1"/>
+        <limit lower="0.0" upper="${PI/2}" effort="${effort}" velocity="${velocity}"/>
+    </joint>
 </robot>

Commit message: todays work

File: src/rain_arm_description/urdf/rain_arm.urdf.xacro (robot description, xacro)
@@ -4,6 +4,13 @@
     <xacro:property name="effort" value="30"/>
     <xacro:property name="velocity" value="10"/>
+    <xacro:macro name="default_inertial" params="mass">
+        <inertial>
+            <mass value="${mass}"/>
+            <inertia ixx="1.0" ixy="0.0" ixz="0.0" iyy="1.0" iyz="0.0" izz="1.0"/>
+        </inertial>
+    </xacro:macro>
     <link name="world"/>
     <link name="base_link">
+        <xacro:default_inertial mass = "1.0"/>
         <visual>
             <origin xyz="-0.5 -0.5 0.0" rpy="0.0 0.0 0.0"/>
@@ -12,4 +19,10 @@
             </geometry>
         </visual>
+        <collision>
+            <origin xyz="-0.5 -0.5 0.0" rpy="0.0 0.0 0.0"/>
+                <geometry>
+                    <mesh filename="package://rain_arm_description/meshes/basement.STL" scale="0.01 0.01 0.01"/>
+                </geometry>
+        </collision>
     </link>
     <joint name="world_base_link" type="fixed">
@@ -19,4 +32,5 @@
     </joint>
     <link name="base_plate">
+        <xacro:default_inertial mass = "0.1"/>
         <visual>
             <origin xyz="-0.39 -0.39 -0.56" rpy="0.0 0.0 0.0"/>
@@ -25,4 +39,10 @@
             </geometry>
         </visual>
+        <collision>
+            <origin xyz="-0.39 -0.39 -0.56" rpy="0.0 0.0 0.0"/>
+            <geometry>
+                <mesh filename="package://rain_arm_description/meshes/base_plate.STL" scale="0.01 0.01 0.01"/>
+            </geometry>
+        </collision>
     </link>
     <joint name="base_link_base_plate" type="revolute">
@@ -34,4 +54,5 @@
     </joint>
     <link name="forward_drive_arm">
+        <xacro:default_inertial mass = "0.1"/>
         <visual>
             <origin rpy="0.0 -${PI/2} ${PI/2}" xyz="0.19 0.06 -0.08"/>
@@ -40,4 +61,10 @@
             </geometry>
         </visual>
+        <collision>
+            <origin rpy="0.0 -${PI/2} ${PI/2}" xyz="0.19 0.06 -0.08"/>
+            <geometry>
+                <mesh filename="package://rain_arm_description/meshes/forward_drive_arm.STL" scale="0.01 0.01 0.01"/>
+            </geometry>
+        </collision>
     </link>
     <joint name="base_plate_forward_drive_arm" type="revolute">
@@ -49,4 +76,5 @@
     </joint>
     <link name="horizontal_arm">
+        <xacro:default_inertial mass = "0.1"/>
         <visual>
             <origin rpy="${PI/2} 0.0 ${PI/2}" xyz="-0.03 -0.4 -0.06"/>
@@ -55,4 +83,10 @@
             </geometry>
         </visual>
+        <collision>
+                <origin rpy="${PI/2} 0.0 ${PI/2}" xyz="-0.03 -0.4 -0.06"/>
+                <geometry>
+                    <mesh filename="package://rain_arm_description/meshes/horizontal_arm.STL" scale="0.01 0.01 0.01"/>
+                </geometry>
+        </collision>
     </link>
     <joint name="forward_drive_arm_horizontal_arm" type="revolute">
@@ -64,4 +98,5 @@
     </joint>
     <link name="claw_base">
+        <xacro:default_inertial mass = "0.05"/>
         <visual>
             <origin xyz="0.0 -0.05 -0.15" rpy="0.0 0.0 ${PI/2}"/>
@@ -70,4 +105,10 @@
             </geometry>
         </visual>
+        <collision>
+            <origin xyz="0.0 -0.05 -0.15" rpy="0.0 0.0 ${PI/2}"/>
+            <geometry>
+                <mesh filename="package://rain_arm_description/meshes/claw_support.STL" scale="0.01 0.01 0.01"/>
+            </geometry>
+        </collision>
     </link>
         <joint name="horizontal_arm_claw_base" type="fixed">
@@ -77,4 +118,5 @@
         </joint>
         <link name="gripper_right">
+            <xacro:default_inertial mass = "0.01"/>
             <visual>
                 <origin xyz="-0.1 0.5 -0.1" rpy="0.0 0.0 -${PI/2}"/>
@@ -83,6 +125,13 @@
                 </geometry>
             </visual>
+            <collision>
+                <origin xyz="-0.1 0.5 -0.1" rpy="0.0 0.0 -${PI/2}"/>
+                <geometry>
+                    <mesh filename="package://rain_arm_description/meshes/right_finger.STL" scale="0.01 0.01 0.01"/>
+                </geometry>
+            </collision>
         </link>
         <link name="gripper_left">
+            <xacro:default_inertial mass = "0.01"/>
             <visual>
                 <origin xyz="-0.04 0.5 -0.1" rpy="0.0 0.0 -${PI/2}"/>
@@ -91,4 +140,10 @@
                 </geometry>
             </visual>
+            <collision>
+                <origin xyz="-0.04 0.5 -0.1" rpy="0.0 0.0 -${PI/2}"/>
+                <geometry>
+                    <mesh filename="package://rain_arm_description/meshes/left_finger.STL" scale="0.01 0.01 0.01"/>
+                </geometry>
+            </collision>
         </link>
     <joint name="claw_base_gripper_right" type="revolute">

Commit message: good morning

File: src/rain_arm_description/urdf/rain_arm.urdf.xacro (robot description, xacro)
@@ -1,4 +1,6 @@
 <?xml version="1.0"?>
 <robot xmlns:xacro="http://www.ros.org/wiki/xacro" name="rain_arm">
+    <xacro:include filename="$(find rain_arm_description)/urdf/rain_arm_gazebo.xacro"/>
+    <xacro:include filename="$(find rain_arm_description)/urdf/rain_arm_ros2_control.xacro"/>
     <xacro:property name="PI" value="3.14159"/>
     <xacro:property name="effort" value="30"/>
@@ -9,4 +11,11 @@
             <inertia ixx="1.0" ixy="0.0" ixz="0.0" iyy="1.0" iyz="0.0" izz="1.0"/>
         </inertial>
+    </xacro:macro>
+    <xacro:macro name = "default_transmission" params = "joint_name">
+        <transmission name="transmission_of_${joint_name}">
+            <plugin>transmission_interface/SimpleTransmission</plugin>
+            <actuator name= "motor_of_${joint_name}" role ="actuator1"></actuator>
+            <joint name="${joint_name}" role="joint1"/>
+        </transmission>
     </xacro:macro>
     <link name="world"/>
@@ -162,3 +171,7 @@
         <limit lower="0.0" upper="${PI/2}" effort="${effort}" velocity="${velocity}"/>
     </joint>
+    <xacro:default_transmission joint_name = "base_link_base_plate"/>
+    <xacro:default_transmission joint_name = "base_plate_forward_drive_arm"/>
+    <xacro:default_transmission joint_name = "claw_base_gripper_right"/>
+    <xacro:default_transmission joint_name = "forward_drive_arm_horizontal_arm"/>
 </robot>

Commit message: i fixed the mimic error

File: src/rain_arm_description/urdf/rain_arm.urdf.xacro (robot description, xacro)
@@ -15,6 +15,8 @@
         <transmission name="transmission_of_${joint_name}">
             <plugin>transmission_interface/SimpleTransmission</plugin>
-            <actuator name= "motor_of_${joint_name}" role ="actuator1"></actuator>
-            <joint name="${joint_name}" role="joint1"/>
+            <actuator name= "motor_of_${joint_name}" role ="actuator1"/>
+            <joint name="${joint_name}" role="joint1">
+                <mechanical_decution>1.0</mechanical_decution>
+            </joint>
         </transmission>
     </xacro:macro>
@@ -156,4 +158,10 @@
             </collision>
         </link>
+    <!-- My fix for the mimic issues (I suffered ooo) -->
+        <joint name="claw_base_gripper_left_mimic" type="fixed">
+            <parent link="world" />
+            <child link="random" />
+          </joint>
+          <link name="random"/>
     <joint name="claw_base_gripper_right" type="revolute">
         <parent link="claw_base"/>
